File: tinyLarson.brd (EAGLE design)
At the start: 57 x 32 mm, 37 parts, among them J1 Ext Bat, U1 ATtiny84A-SSU, U2 MCP1640D

Commit message: Add images.
Parts:
- C2: value 10uF -> 4.7uF
- D0, D1, D2, D3, D4, D5, D6: device _jc:M0805 -> _jc:D0805A
- D7: device _jc:M0805 -> _jc:D0805
- LOGO2: value OSHW_LOGO_10MILX0200-NT -> OSHW_LOGO_8MILX0100-NT; device ohw-logo:OSHW_10X200_NOTEXT -> ohw-logo:OSHW_8X100_NOTEXT
- moved LOGO1 61.2 mm to (8.60, 2.30)
- moved LOGO2 35.0 mm to (9.50, 17.0)
- moved R0 9.22 mm to (49.5, 29.0), flipped to the bottom, turned to 270 degrees
- moved R1 3.04 mm to (43.5, 29.0), flipped to the bottom, turned to 270 degrees
- moved R2 3.04 mm to (37.5, 29.0), flipped to the bottom, turned to 270 degrees
- moved R3 3.04 mm to (31.5, 29.0), flipped to the bottom, turned to 270 degrees
- moved R4 3.04 mm to (25.5, 29.0), flipped to the bottom, turned to 270 degrees
- moved R5 3.04 mm to (19.5, 29.0), flipped to the bottom, turned to 270 degrees
- moved R6 3.04 mm to (13.5, 29.0), flipped to the bottom, turned to 270 degrees
- moved R7 3.04 mm to (7.50, 29.0), flipped to the bottom, turned to 270 degrees
- moved D8 0.71 mm to (43.5, 20.5)
- moved D0 0.50 mm to (49.5, 29.0), turned to 90 degrees
- moved D1 0.50 mm to (43.5, 29.0), turned to 90 degrees
- moved D2 0.50 mm to (37.5, 29.0), turned to 90 degrees
- moved D3 0.50 mm to (31.5, 29.0), turned to 90 degrees
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Connections:
- net GND: now also D0.K, D1.K, D2.K, D3.K, D4.K, D5.K, D6.K, D7.K; no longer D0.2, D1.2, D2.2, D3.2, D4.2, D5.2, D6.2, D7.2
- net N$10: now also D6.A; no longer D6.1
- net N$12: now also D7.A; no longer D7.1
- net N$3: now also D0.A; no longer D0.1
- net N$4: now also D1.A; no longer D1.1
- net N$5: now also D2.A; no longer D2.1
- net N$6: now also D3.A; no longer D3.1
- net N$8: now also D4.A; no longer D4.1
- net N$9: now also D5.A; no longer D5.1
Routing:
- net N$3: track 9.98 -> 4.46 mm, vias 0 -> 1
- net PA7: track 31.9 -> 36.9 mm, vias 2 -> 1
- net MOSI: track 51.9 -> 56.0 mm, vias 3 -> 2
- net MISO: track 48.2 -> 50.7 mm, vias 3 -> 2
- net PB2: track 16.1 -> 13.9 mm
- net PA0: track 43.7 -> 45.5 mm, vias 2 -> 1
- net SCK: track 48.6 -> 50.3 mm, vias 2 -> 1
- net N$6: track 3.00 -> 4.46 mm, vias 0 -> 1
- net N$5: track 3.00 -> 4.46 mm, vias 0 -> 1
- net N$4: track 3.00 -> 4.46 mm, vias 0 -> 1
- net N$9: track 3.00 -> 4.46 mm, vias 0 -> 1
- net N$8: track 3.00 -> 4.46 mm, vias 0 -> 1
- net N$12: track 3.00 -> 4.46 mm, vias 0 -> 1
- net N$10: track 3.00 -> 4.46 mm, vias 0 -> 1
- net N$11: track 25.1 -> 26.5 mm
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Other:
- board text added: "+"
- board text added: "-"
- board text added: "CC BY-SA 4.0 jc 0519"
- board text added: "CC BY-SA 4.0 jc 0519 open source bit.ly/tnylrsn"
- board text added: "SELECT"
- board text added: "open source bit.ly/tnylrsn"
- board text added: "tinyLarson v1.0"
- board text removed: "CC BY-SA 4.0"
- board text removed: "CC BY-SA 4.0 jc 0118"
- board text removed: "jc 0118"
- board text removed: "open source goo.gl/LtKUka"
- board text removed: "tinyTimer v1.0"
