File: tinyLarson.sch (EAGLE design)
At the start: 37 parts, among them J1 Ext Bat, U1 ATtiny84A-SSU, U2 MCP1640D

Commit message: Add images.
Parts:
- C2: value 10uF -> 4.7uF
- D0, D1, D2, D3, D4, D5, D6: device _jc:LEDM0805 -> _jc:LEDD0805A
- D7: device _jc:LEDM0805 -> _jc:LEDD0805
- LOGO2: value OSHW_LOGO_10MILX0200-NT -> OSHW_LOGO_8MILX0100-NT; device ohw-logo:OSHW_LOGO_10MILX0200-NT -> ohw-logo:OSHW_LOGO_8MILX0100-NT
Changed lines of the file:
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@@
 <grid distance="0.1" unitdist="inch" unit="inch" style="lines" multiple="1" display="no" altdistance="0.01" altunitdist="inch" altunit="inch"/>
 <layers>
-<layer number="1" name="Top" color="4" fill="1" visible="yes" active="no"/>
-<layer number="16" name="Bottom" color="1" fill="1" visible="yes" active="no"/>
-<layer number="17" name="Pads" color="2" fill="1" visible="yes" active="no"/>
-<layer number="18" name="Vias" color="2" fill="1" visible="yes" active="no"/>
-<layer number="19" name="Unrouted" color="6" fill="1" visible="yes" active="no"/>
-<layer number="20" name="Dimension" color="15" fill="1" visible="yes" active="no"/>
-<layer number="21" name="tPlace" color="7" fill="1" visible="yes" active="no"/>
-<layer number="22" name="bPlace" color="7" fill="1" visible="yes" active="no"/>
-<layer number="23" name="tOrigins" color="15" fill="1" visible="yes" active="no"/>
-<layer number="24" name="bOrigins" color="15" fill="1" visible="yes" active="no"/>
-<layer number="25" name="tNames" color="7" fill="1" visible="yes" active="no"/>
-<layer number="26" name="bNames" color="7" fill="1" visible="yes" active="no"/>
-<layer number="27" name="tValues" color="7" fill="1" visible="yes" active="no"/>
-<layer number="28" name="bValues" color="7" fill="1" visible="yes" active="no"/>
+<layer number="1" name="Top" color="4" fill="1" visible="no" active="no"/>
+<layer number="16" name="Bottom" color="1" fill="1" visible="no" active="no"/>
+<layer number="17" name="Pads" color="2" fill="1" visible="no" active="no"/>
+<layer number="18" name="Vias" color="2" fill="1" visible="no" active="no"/>
+<layer number="19" name="Unrouted" color="6" fill="1" visible="no" active="no"/>
+<layer number="20" name="Dimension" color="15" fill="1" visible="no" active="no"/>
+<layer number="21" name="tPlace" color="7" fill="1" visible="no" active="no"/>
+<layer number="22" name="bPlace" color="7" fill="1" visible="no" active="no"/>
+<layer number="23" name="tOrigins" color="15" fill="1" visible="no" active="no"/>
+<layer number="24" name="bOrigins" color="15" fill="1" visible="no" active="no"/>
+<layer number="25" name="tNames" color="7" fill="1" visible="no" active="no"/>
+<layer number="26" name="bNames" color="7" fill="1" visible="no" active="no"/>
+<layer number="27" name="tValues" color="7" fill="1" visible="no" active="no"/>
+<layer number="28" name="bValues" color="7" fill="1" visible="no" active="no"/>
 <layer number="29" name="tStop" color="7" fill="3" visible="no" active="no"/>
 <layer number="30" name="bStop" color="7" fill="6" visible="no" active="no"/>
@@
 <layer number="35" name="tGlue" color="7" fill="4" visible="no" active="no"/>
 <layer number="36" name="bGlue" color="7" fill="5" visible="no" active="no"/>
-<layer number="37" name="tTest" color="7" fill="1" visible="yes" active="no"/>
-<layer number="38" name="bTest" color="7" fill="1" visible="yes" active="no"/>
+<layer number="37" name="tTest" color="7" fill="1" visible="no" active="no"/>
+<layer number="38" name="bTest" color="7" fill="1" visible="no" active="no"/>
 <layer number="39" name="tKeepout" color="4" fill="11" visible="no" active="no"/>
 <layer number="40" name="bKeepout" color="1" fill="11" visible="no" active="no"/>
@@
 <layer number="44" name="Drills" color="7" fill="1" visible="no" active="no"/>
 <layer number="45" name="Holes" color="7" fill="1" visible="no" active="no"/>
-<layer number="46" name="Milling" color="3" fill="1" visible="yes" active="no"/>
-<layer number="47" name="Measures" color="7" fill="1" visible="yes" active="no"/>
-<layer number="48" name="Document" color="7" fill="1" visible="yes" active="no"/>
-<layer number="49" name="Reference" color="7" fill="1" visible="yes" active="no"/>
-<layer number="50" name="dxf" color="7" fill="1" visible="yes" active="no"/>
-<layer number="51" name="tDocu" color="7" fill="1" visible="yes" active="no"/>
-<layer number="52" name="bDocu" color="7" fill="1" visible="yes" active="no"/>
-<layer number="53" name="tGND_GNDA" color="7" fill="9" visible="yes" active="no"/>
-<layer number="54" name="bGND_GNDA" color="1" fill="9" visible="yes" active="no"/>
-<layer number="56" name="wert" color="7" fill="1" visible="yes" active="no"/>
-<layer number="57" name="tCAD" color="7" fill="1" visible="yes" active="no"/>
-<layer number="59" name="tCarbon" color="7" fill="1" visible="yes" active="no"/>
-<layer number="60" name="bCarbon" color="7" fill="1" visible="yes" active="no"/>
+<layer number="46" name="Milling" color="3" fill="1" visible="no" active="no"/>
+<layer number="47" name="Measures" color="7" fill="1" visible="no" active="no"/>
+<layer number="48" name="Document" color="7" fill="1" visible="no" active="no"/>
+<layer number="49" name="Reference" color="7" fill="1" visible="no" active="no"/>
+<layer number="50" name="dxf" color="7" fill="1" visible="no" active="no"/>
+<layer number="51" name="tDocu" color="7" fill="1" visible="no" active="no"/>
+<layer number="52" name="bDocu" color="7" fill="1" visible="no" active="no"/>
+<layer number="53" name="tGND_GNDA" color="7" fill="9" visible="no" active="no"/>
+<layer number="54" name="bGND_GNDA" color="1" fill="9" visible="no" active="no"/>
+<layer number="56" name="wert" color="7" fill="1" visible="no" active="no"/>
+<layer number="57" name="tCAD" color="7" fill="1" visible="no" active="no"/>
+<layer number="59" name="tCarbon" color="7" fill="1" visible="no" active="no"/>
+<layer number="60" name="bCarbon" color="7" fill="1" visible="no" active="no"/>
 <layer number="90" name="Modules" color="5" fill="1" visible="yes" active="yes"/>
 <layer number="91" name="Nets" color="2" fill="1" visible="yes" active="yes"/>
@@
 </part>
 <part name="GND6" library="supply1" deviceset="GND" device=""/>
-<part name="C2" library="_jc" deviceset="C-US" device="M0805" value="10uF"/>
+<part name="C2" library="_jc" deviceset="C-US" device="M0805" value="4.7uF"/>
 <part name="C3" library="_jc" deviceset="C-US" device="M0805" value="10uF"/>
 <part name="GND9" library="supply1" deviceset="GND" device=""/>
@@
 <part name="GND2" library="supply1" deviceset="GND" device=""/>
 <part name="GND7" library="supply1" deviceset="GND" device=""/>
-<part name="LOGO2" library="ohw-logo" deviceset="OSHW_LOGO_10MIL" device="X0200-NT" value="OSHW_LOGO_10MILX0200-NT"/>
 <part name="SJ1" library="jumper" deviceset="SJ" device="" value="5V"/>
 <part name="R12" library="_jc" deviceset="R-US_" device="M0805" value="249K"/>
@@
 <part name="GND12" library="supply1" deviceset="GND" device=""/>
 <part name="R0" library="_jc" deviceset="R-US_" device="M0805" value="1K"/>
-<part name="D0" library="_jc" deviceset="LED" device="M0805" value="Yel">
+<part name="D0" library="_jc" deviceset="LED" device="D0805A" value="Yel">
 <attribute name="MFR" value="Lite-On"/>
 <attribute name="MFR-PART-NO" value="LTST-C171KYKT"/>
 </part>
 <part name="R1" library="_jc" deviceset="R-US_" device="M0805" value="1K"/>
-<part name="D1" library="_jc" deviceset="LED" device="M0805" value="Yel">
+<part name="D1" library="_jc" deviceset="LED" device="D0805A" value="Yel">
 <attribute name="MFR" value="Lite-On"/>
 <attribute name="MFR-PART-NO" value="LTST-C171KYKT"/>
 </part>
 <part name="R2" library="_jc" deviceset="R-US_" device="M0805" value="1K"/>
-<part name="D2" library="_jc" deviceset="LED" device="M0805" value="Yel">
+<part name="D2" library="_jc" deviceset="LED" device="D0805A" value="Yel">
 <attribute name="MFR" value="Lite-On"/>
 <attribute name="MFR-PART-NO" value="LTST-C171KYKT"/>
 </part>
 <part name="R3" library="_jc" deviceset="R-US_" device="M0805" value="1K"/>
-<part name="D3" library="_jc" deviceset="LED" device="M0805" value="Yel">
+<part name="D3" library="_jc" deviceset="LED" device="D0805A" value="Yel">
 <attribute name="MFR" value="Lite-On"/>
 <attribute name="MFR-PART-NO" value="LTST-C171KYKT"/>
 </part>
 <part name="R4" library="_jc" deviceset="R-US_" device="M0805" value="1K"/>
-<part name="D4" library="_jc" deviceset="LED" device="M0805" value="Yel">
+<part name="D4" library="_jc" deviceset="LED" device="D0805A" value="Yel">
 <attribute name="MFR" value="Lite-On"/>
 <attribute name="MFR-PART-NO" value="LTST-C171KYKT"/>
 </part>
 <part name="R5" library="_jc" deviceset="R-US_" device="M0805" value="1K"/>
-<part name="D5" library="_jc" deviceset="LED" device="M0805" value="Yel">
+<part name="D5" library="_jc" deviceset="LED" device="D0805A" value="Yel">
 <attribute name="MFR" value="Lite-On"/>
 <attribute name="MFR-PART-NO" value="LTST-C171KYKT"/>
 </part>
 <part name="R6" library="_jc" deviceset="R-US_" device="M0805" value="1K"/>
-<part name="D6" library="_jc" deviceset="LED" device="M0805" value="Yel">
+<part name="D6" library="_jc" deviceset="LED" device="D0805A" value="Yel">
 <attribute name="MFR" value="Lite-On"/>
 <attribute name="MFR-PART-NO" value="LTST-C171KYKT"/>
 </part>
 <part name="R7" library="_jc" deviceset="R-US_" device="M0805" value="1K"/>
-<part name="D7" library="_jc" deviceset="LED" device="M0805" value="Yel">
+<part name="D7" library="_jc" deviceset="LED" device="D0805" value="Yel">
 <attribute name="MFR" value="Lite-On"/>
 <attribute name="MFR-PART-NO" value="LTST-C171KYKT"/>
@@
 <part name="J1" library="_jc" deviceset="OST-TB-2" device="3.5MM" value="Ext Bat"/>
 <part name="GND8" library="supply1" deviceset="GND" device=""/>
+<part name="LOGO2" library="ohw-logo" deviceset="OSHW_LOGO_8MIL" device="X0100-NT" value="OSHW_LOGO_8MILX0100-NT"/>
 </parts>
 <sheets>
@@
 </instance>
 <instance part="GND7" gate="1" x="137.16" y="116.84"/>
-<instance part="LOGO2" gate="G$1" x="68.58" y="17.78"/>
 <instance part="SJ1" gate="1" x="104.14" y="43.18" smashed="yes" rot="R90">
 <attribute name="NAME" x="107.442" y="37.846" size="1.778" layer="95" rot="R90"/>
@@
 <instance part="J1" gate="G$1" x="22.86" y="60.96"/>
 <instance part="GND8" gate="1" x="30.48" y="35.56"/>
+<instance part="LOGO2" gate="G$1" x="68.58" y="17.78"/>
 </instances>
 <busses>

Commit message: Update schematic document number.
Other:
- note added: "MIL-TFD-41"
Changed lines of the file:
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@@
 <?xml version="1.0" encoding="utf-8"?>
 <!DOCTYPE eagle SYSTEM "eagle.dtd">
-<eagle version="7.5.0">
+<eagle version="9.6.2">
 <drawing>
 <settings>
 <setting alwaysvectorfont="yes"/>
+<setting keepoldvectorfont="yes"/>
 <setting verticaltext="up"/>
 </settings>
@@
 <text x="175.768" y="24.638" size="2.54" layer="94" ratio="12">by Jack Christensen</text>
 <text x="262.128" y="6.858" size="2.54" layer="94" ratio="12">v1.0</text>
+<text x="191.008" y="6.858" size="2.54" layer="94" ratio="12">MIL-TFD-41</text>
 </plain>
 <instances>
-<instance part="FRAME1" gate="G$1" x="0" y="0"/>
-<instance part="FRAME1" gate="G$2" x="172.72" y="0"/>
-<instance part="GND1" gate="1" x="40.64" y="35.56"/>
+<instance part="FRAME1" gate="G$1" x="0" y="0" smashed="yes"/>
+<instance part="FRAME1" gate="G$2" x="172.72" y="0" smashed="yes">
+<attribute name="LAST_DATE_TIME" x="185.42" y="1.27" size="2.54" layer="94" font="vector"/>
+<attribute name="SHEET" x="259.08" y="1.27" size="2.54" layer="94" font="vector"/>
+<attribute name="DRAWING_NAME" x="190.5" y="19.05" size="2.54" layer="94" font="vector"/>
+</instance>
+<instance part="GND1" gate="1" x="40.64" y="35.56" smashed="yes">
+<attribute name="VALUE" x="38.1" y="33.02" size="1.778" layer="96"/>
+</instance>
 <instance part="U2" gate="G$1" x="78.74" y="63.5" smashed="yes">
 <attribute name="NAME" x="71.12" y="53.34" size="1.778" layer="94"/>
@@
 <attribute name="VALUE" x="93.98" y="33.02" size="1.778" layer="96"/>
 </instance>
-<instance part="P+3" gate="VCC" x="111.76" y="76.2"/>
-<instance part="GND3" gate="1" x="162.56" y="35.56"/>
-<instance part="P+5" gate="VCC" x="162.56" y="58.42"/>
-<instance part="B1" gate="G$1" x="40.64" y="53.34">
+<instance part="P+3" gate="VCC" x="111.76" y="76.2" smashed="yes">
+<attribute name="VALUE" x="109.22" y="73.66" size="1.778" layer="96" rot="R90"/>
+</instance>
+<instance part="GND3" gate="1" x="162.56" y="35.56" smashed="yes">
+<attribute name="VALUE" x="160.02" y="33.02" size="1.778" layer="96"/>
+</instance>
+<instance part="P+5" gate="VCC" x="162.56" y="58.42" smashed="yes">
+<attribute name="VALUE" x="160.02" y="55.88" size="1.778" layer="96" rot="R90"/>
+</instance>
+<instance part="B1" gate="G$1" x="40.64" y="53.34" smashed="yes">
 <attribute name="MFR" x="40.64" y="53.34" size="1.778" layer="96" display="off"/>
 <attribute name="MFR-PART-NO" x="40.64" y="53.34" size="1.778" layer="96" display="off"/>
-</instance>
-<instance part="ICSP" gate="G$1" x="149.86" y="45.72"/>
-<instance part="U1" gate="G$1" x="48.26" y="129.54"/>
+<attribute name="NAME" x="45.72" y="63.5" size="1.778" layer="95"/>
+<attribute name="VALUE" x="45.72" y="60.96" size="1.778" layer="96"/>
+</instance>
+<instance part="ICSP" gate="G$1" x="149.86" y="45.72" smashed="yes">
+<attribute name="NAME" x="145.542" y="54.102" size="1.778" layer="95"/>
+<attribute name="VALUE" x="145.796" y="35.56" size="1.778" layer="96"/>
+</instance>
+<instance part="U1" gate="G$1" x="48.26" y="129.54" smashed="yes">
+<attribute name="NAME" x="48.26" y="162.56" size="1.778" layer="95"/>
+<attribute name="VALUE" x="58.42" y="162.56" size="1.778" layer="96"/>
+</instance>
 <instance part="P+2" gate="VCC" x="30.48" y="175.26" smashed="yes">
 <attribute name="VALUE" x="27.94" y="172.72" size="1.778" layer="96" rot="R90"/>
@@
 <attribute name="VALUE" x="35.56" y="121.92" size="1.778" layer="96"/>
 </instance>
-<instance part="S1" gate="1" x="45.72" y="99.06">
+<instance part="S1" gate="1" x="45.72" y="99.06" smashed="yes">
 <attribute name="MFR" x="45.72" y="99.06" size="1.778" layer="96" display="off"/>
 <attribute name="MFR-PART-NO" x="45.72" y="99.06" size="1.778" layer="96" display="off"/>
-</instance>
-<instance part="LOGO1" gate="G$1" x="55.88" y="17.78"/>
+<attribute name="NAME" x="39.37" y="96.52" size="1.778" layer="95" rot="R90"/>
+<attribute name="VALUE" x="41.91" y="102.235" size="1.778" layer="96" rot="R90"/>
+</instance>
+<instance part="LOGO1" gate="G$1" x="55.88" y="17.78" smashed="yes"/>
 <instance part="GND2" gate="1" x="45.72" y="88.9" smashed="yes">
 <attribute name="VALUE" x="43.18" y="86.36" size="1.778" layer="96"/>
 </instance>
-<instance part="GND7" gate="1" x="137.16" y="116.84"/>
+<instance part="GND7" gate="1" x="137.16" y="116.84" smashed="yes">
+<attribute name="VALUE" x="134.62" y="114.3" size="1.778" layer="96"/>
+</instance>
 <instance part="SJ1" gate="1" x="104.14" y="43.18" smashed="yes" rot="R90">
 <attribute name="NAME" x="107.442" y="37.846" size="1.778" layer="95" rot="R90"/>
@@
 <attribute name="VALUE" x="93.218" y="46.99" size="1.778" layer="96" rot="R270"/>
 </instance>
-<instance part="JP1" gate="G$1" x="20.32" y="99.06"/>
-<instance part="S2" gate="1" x="20.32" y="139.7">
+<instance part="JP1" gate="G$1" x="20.32" y="99.06" smashed="yes">
+<attribute name="VALUE" x="17.78" y="93.98" size="1.778" layer="96"/>
+<attribute name="NAME" x="17.78" y="104.902" size="1.778" layer="95"/>
+</instance>
+<instance part="S2" gate="1" x="20.32" y="139.7" smashed="yes">
 <attribute name="MFR" x="20.32" y="139.7" size="1.778" layer="96" display="off"/>
 <attribute name="MFR-PART-NO" x="20.32" y="139.7" size="1.778" layer="96" display="off"/>
+<attribute name="NAME" x="13.97" y="137.16" size="1.778" layer="95" rot="R90"/>
+<attribute name="VALUE" x="16.51" y="142.875" size="1.778" layer="96" rot="R90"/>
 </instance>
 <instance part="GND11" gate="1" x="20.32" y="124.46" smashed="yes">
 <attribute name="VALUE" x="17.78" y="121.92" size="1.778" layer="96"/>
 </instance>
-<instance part="GND12" gate="1" x="27.94" y="88.9"/>
+<instance part="GND12" gate="1" x="27.94" y="88.9" smashed="yes">
+<attribute name="VALUE" x="25.4" y="86.36" size="1.778" layer="96"/>
+</instance>
 <instance part="R0" gate="G$1" x="167.64" y="132.08" smashed="yes" rot="R270">
 <attribute name="NAME" x="169.1386" y="135.89" size="1.778" layer="95" rot="R270"/>
@@
 <attribute name="MFR-PART-NO" x="104.14" y="124.46" size="1.778" layer="96" display="off"/>
 </instance>
-<instance part="J1" gate="G$1" x="22.86" y="60.96"/>
-<instance part="GND8" gate="1" x="30.48" y="35.56"/>
-<instance part="LOGO2" gate="G$1" x="68.58" y="17.78"/>
+<instance part="J1" gate="G$1" x="22.86" y="60.96" smashed="yes">
+<attribute name="NAME" x="17.78" y="66.802" size="1.778" layer="95"/>
+<attribute name="VALUE" x="17.018" y="55.88" size="1.778" layer="96" rot="R90"/>
+</instance>
+<instance part="GND8" gate="1" x="30.48" y="35.56" smashed="yes">
+<attribute name="VALUE" x="27.94" y="33.02" size="1.778" layer="96"/>
+</instance>
+<instance part="LOGO2" gate="G$1" x="68.58" y="17.78" smashed="yes"/>
 </instances>
 <busses>
